File: gw1ns2c-board.sch (KiCad schematic (older format))
At the start: 39 parts, among them J1 USB_B_Micro, J2 Conn_01x20, J3 Conn_01x20, SW1 SW_Push, U1 STM32F042F6Px, U2 GW1NS-2CQN48, U3 TPS73101DBV, U4 MIC5504-3.3YM5, U5 TPS73101DBV

Commit message: Add post-assembly notes
Parts:
- R10: value 56.2k -> 68k
- R9: value 28k -> 33k
Other:
- note added: "According to the datasheet,\nrecommended resistor values\nare 28k / 56.2k, but 33k / 68k\nalso works fine.\nAnyway, this power supply\nis not used with UX chips."
- note added: "Deviation: on a board 4.3k\nis used instead of 4.7k"
Changed lines of the file:
@@
 U 1 1 60128EA8
 P 6600 5150
-F 0 "D2" V 6646 4820 50  0000 R CNN
-F 1 "LED_RGBA" V 6555 4820 50  0000 R CNN
+F 0 "D2" H 6600 4775 50  0000 C CNN
+F 1 "LED_RGBA" H 6600 4684 50  0000 C CNN
 F 2 "LED_SMD:LED_LiteOn_LTST-C19HE1WT" H 6600 5100 50  0001 C CNN
 F 3 "~" H 6600 5100 50  0001 C CNN
@@
 P 2350 6850
 F 0 "R9" H 2291 6804 50  0000 R CNN
-F 1 "28k" H 2291 6895 50  0000 R CNN
+F 1 "33k" H 2291 6895 50  0000 R CNN
 F 2 "Resistor_SMD:R_0603_1608Metric" H 2350 6850 50  0001 C CNN
 F 3 "~" H 2350 6850 50  0001 C CNN
@@
 P 2350 7050
 F 0 "R10" H 2291 7004 50  0000 R CNN
-F 1 "56.2k" H 2291 7095 50  0000 R CNN
+F 1 "68k" H 2291 7095 50  0000 R CNN
 F 2 "Resistor_SMD:R_0603_1608Metric" H 2350 7050 50  0001 C CNN
 F 3 "~" H 2350 7050 50  0001 C CNN
@@
 	1    0    0    -1
 $EndComp
+Text Notes 1950 7700 0    50   ~ 0
+According to the datasheet,\nrecommended resistor values\nare 28k / 56.2k, but 33k / 68k\nalso works fine.\nAnyway, this power supply\nis not used with UX chips.
+Text Notes 550  4600 0    50   ~ 0
+Deviation: on a board 4.3k\nis used instead of 4.7k
 $EndSCHEMATC
